File: EVBuild/EVBuild.kicad_sch (KiCad schematic)
At the start: 5 parts, among them J1 Spark Max PWM, U1 ESP32-S3-WROOM-2

Commit message: the stuff
Parts:
- added LSF1: ~, symbol LSF0102:LSF0102
- added NCP1: ~, symbol NCP551:NCP551
Connections:
- net GND: now reaches U1.1 (GND), U1.40 (GND), U1.41 (GND)
- net GND: now also FlyDragon1. (VCC), LSF1.1 (GND)
Other:
- note removed: "Logic Shifter https://www.ti.com/lit/ds/symlink/lsf0102.pdf?HQS=dis-dk-null-digikeymode-dsf-pf-null-wwe&ts=1737043697636&ref_url=https%253A%252F%252Fwww.ti.com%252Fgeneral%252Fdocs%252Fsuppproductinfo.tsp%253FdistId%253D10%2526gotoUrl%253Dhttps%253A%252F%252Fwww.ti.com%252Flit%252Fgpn%252Flsf0102 Voltage Regulator: 12-3.3V"
- moved on the sheet: FlyDragon1, J1
Changed lines of the file:
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@@
 (kicad_sch (version 20230121) (generator eeschema)
   (paper "A4")
-  (text "Logic Shifter\nhttps://www.ti.com/lit/ds/symlink/lsf0102.pdf?HQS=dis-dk-null-digikeymode-dsf-pf-null-wwe&ts=1737043697636&ref_url=https%253A%252F%252Fwww.ti.com%252Fgeneral%252Fdocs%252Fsuppproductinfo.tsp%253FdistId%253D10%2526gotoUrl%253Dhttps%253A%252F%252Fwww.ti.com%252Flit%252Fgpn%252Flsf0102\nVoltage Regulator: 12-3.3V"
-    (at 209.55 121.92 0)
-    (effects (font (size 1.27 1.27)) (justify left bottom))
+  (wire (pts (xy 219.71 76.2) (xy 220.98 76.2))
+    (stroke (width 0) (type default))
+  )
+  (wire (pts (xy 220.98 76.2) (xy 220.98 77.47))
+    (stroke (width 0) (type default))
   )
   (symbol (lib_id "RF_Module:ESP32-S3-WROOM-2") (at 121.92 85.09 0) (unit 1)
@@
     )
   )
-  (symbol (lib_id "Connector:Conn_01x04_Pin") (at 176.53 99.06 0) (unit 1)
-    (in_bom yes) (on_board yes) (dnp no) (fields_autoplaced)
-    (property "Reference" "J1" (at 177.165 91.44 0)
-      (effects (font (size 1.27 1.27)))
-    )
-    (property "Value" "Spark Max PWM" (at 177.165 93.98 0)
-      (effects (font (size 1.27 1.27)))
-    )
-    (property "Footprint" "Connector_JST:JST_PH_S4B-PH-K_1x04_P2.00mm_Horizontal" (at 176.53 99.06 0)
-      (effects (font (size 1.27 1.27)) hide)
-    )
-    (property "Datasheet" "~" (at 176.53 99.06 0)
+  (symbol (lib_id "power:GND") (at 252.73 62.23 0) (unit 1)
+    (in_bom yes) (on_board yes) (dnp no) (fields_autoplaced)
+    (property "Reference" "#PWR02" (at 252.73 68.58 0)
+      (effects (font (size 1.27 1.27)) hide)
+    )
+    (property "Value" "GND" (at 252.73 67.31 0)
+      (effects (font (size 1.27 1.27)))
+    )
+    (property "Footprint" "" (at 252.73 62.23 0)
+      (effects (font (size 1.27 1.27)) hide)
+    )
+    (property "Datasheet" "" (at 252.73 62.23 0)
+      (effects (font (size 1.27 1.27)) hide)
+    )
+    (pin "1")
+    (instances
+      (project "EVBuild"
+        (path "/2997cb29-a416-41db-a9e8-1a576f951325"
+          (reference "#PWR02") (unit 1)
+        )
+      )
+    )
+  )
+  (symbol (lib_id "LSF0102:LSF0102") (at 255.27 59.69 0) (unit 1)
+    (in_bom yes) (on_board yes) (dnp no) (fields_autoplaced)
+    (property "Reference" "LSF1" (at 254.635 44.45 0)
+      (effects (font (size 1.27 1.27)))
+    )
+    (property "Value" "~" (at 240.03 66.04 0)
+      (effects (font (size 1.27 1.27)))
+    )
+    (property "Footprint" "" (at 240.03 66.04 0)
+      (effects (font (size 1.27 1.27)) hide)
+    )
+    (property "Datasheet" "" (at 240.03 66.04 0)
+      (effects (font (size 1.27 1.27)) hide)
+    )
+    (pin "3")
+    (pin "6")
+    (pin "5")
+    (pin "1")
+    (pin "2")
+    (pin "4")
+    (pin "7")
+    (pin "8")
+    (instances
+      (project "EVBuild"
+        (path "/2997cb29-a416-41db-a9e8-1a576f951325"
+          (reference "LSF1") (unit 1)
+        )
+      )
+    )
+  )
+  (symbol (lib_id "power:GND") (at 220.98 77.47 0) (unit 1)
+    (in_bom yes) (on_board yes) (dnp no) (fields_autoplaced)
+    (property "Reference" "#PWR03" (at 220.98 83.82 0)
+      (effects (font (size 1.27 1.27)) hide)
+    )
+    (property "Value" "GND" (at 220.98 82.55 0)
+      (effects (font (size 1.27 1.27)))
+    )
+    (property "Footprint" "" (at 220.98 77.47 0)
+      (effects (font (size 1.27 1.27)) hide)
+    )
+    (property "Datasheet" "" (at 220.98 77.47 0)
+      (effects (font (size 1.27 1.27)) hide)
+    )
+    (pin "1")
+    (instances
+      (project "EVBuild"
+        (path "/2997cb29-a416-41db-a9e8-1a576f951325"
+          (reference "#PWR03") (unit 1)
+        )
+      )
+    )
+  )
+  (symbol (lib_id "Connector:Conn_01x04_Pin") (at 231.14 50.8 0) (unit 1)
+    (in_bom yes) (on_board yes) (dnp no) (fields_autoplaced)
+    (property "Reference" "J1" (at 231.775 43.18 0)
+      (effects (font (size 1.27 1.27)))
+    )
+    (property "Value" "Spark Max PWM" (at 231.775 45.72 0)
+      (effects (font (size 1.27 1.27)))
+    )
+    (property "Footprint" "Connector_JST:JST_PH_S4B-PH-K_1x04_P2.00mm_Horizontal" (at 231.14 50.8 0)
+      (effects (font (size 1.27 1.27)) hide)
+    )
+    (property "Datasheet" "~" (at 231.14 50.8 0)
       (effects (font (size 1.27 1.27)) hide)
     )
@@
     )
   )
-  (symbol (lib_id "BMI270:BMI270") (at 180.34 52.07 0) (unit 1)
-    (in_bom yes) (on_board yes) (dnp no) (fields_autoplaced)
-    (property "Reference" "U2" (at 183.8041 36.83 0)
-      (effects (font (size 1.27 1.27)) (justify left))
-    )
-    (property "Value" "~" (at 189.23 50.8 0)
-      (effects (font (size 1.27 1.27)))
-    )
-    (property "Footprint" "Package_LGA:Bosch_LGA-14_3x2.5mm_P0.5mm" (at 180.34 83.82 0)
-      (effects (font (size 1.27 1.27)) hide)
-    )
-    (property "Datasheet" "https://www.bosch-sensortec.com/media/boschsensortec/downloads/datasheets/bst-bmi270-ds000.pdf" (at 180.34 86.36 0)
+  (symbol (lib_id "BMI270:BMI270") (at 38.1 46.99 0) (unit 1)
+    (in_bom yes) (on_board yes) (dnp no) (fields_autoplaced)
+    (property "Reference" "U2" (at 41.5641 31.75 0)
+      (effects (font (size 1.27 1.27)) (justify left) hide)
+    )
+    (property "Value" "~" (at 46.99 45.72 0)
+      (effects (font (size 1.27 1.27)))
+    )
+    (property "Footprint" "Package_LGA:Bosch_LGA-14_3x2.5mm_P0.5mm" (at 38.1 78.74 0)
+      (effects (font (size 1.27 1.27)) hide)
+    )
+    (property "Datasheet" "https://www.bosch-sensortec.com/media/boschsensortec/downloads/datasheets/bst-bmi270-ds000.pdf" (at 38.1 81.28 0)
       (effects (font (size 1.27 1.27)) hide)
     )
@@
     )
   )
-  (symbol (lib_id "0.96InchOLED:0.96_Inch_OLED") (at 179.07 143.51 0) (unit 1)
-    (in_bom yes) (on_board yes) (dnp no) (fields_autoplaced)
-    (property "Reference" "U3" (at 196.85 145.2908 0)
-      (effects (font (size 1.27 1.27)) (justify left))
-    )
-    (property "Value" "~" (at 168.91 146.05 0)
-      (effects (font (size 1.27 1.27)))
-    )
-    (property "Footprint" "Connector_PinHeader_2.54mm:PinHeader_1x04_P2.54mm_Vertical" (at 168.91 146.05 0)
-      (effects (font (size 1.27 1.27)) hide)
-    )
-    (property "Datasheet" "" (at 168.91 146.05 0)
+  (symbol (lib_id "0.96InchOLED:0.96_Inch_OLED") (at 64.77 44.45 0) (unit 1)
+    (in_bom yes) (on_board yes) (dnp no) (fields_autoplaced)
+    (property "Reference" "U3" (at 82.55 46.2308 0)
+      (effects (font (size 1.27 1.27)) (justify left) hide)
+    )
+    (property "Value" "~" (at 54.61 46.99 0)
+      (effects (font (size 1.27 1.27)))
+    )
+    (property "Footprint" "Connector_PinHeader_2.54mm:PinHeader_1x04_P2.54mm_Vertical" (at 54.61 46.99 0)
+      (effects (font (size 1.27 1.27)) hide)
+    )
+    (property "Datasheet" "" (at 54.61 46.99 0)
       (effects (font (size 1.27 1.27)) hide)
     )
@@
     )
   )
-  (symbol (lib_id "FlyDragon:FlyDragon") (at 181.61 123.19 0) (unit 1)
-    (in_bom yes) (on_board yes) (dnp no) (fields_autoplaced)
-    (property "Reference" "FlyDragon1" (at 179.705 113.03 0)
-      (effects (font (size 1.27 1.27)))
-    )
-    (property "Value" "~" (at 172.72 124.46 0)
-      (effects (font (size 1.27 1.27)))
-    )
-    (property "Footprint" "" (at 172.72 124.46 0)
-      (effects (font (size 1.27 1.27)) hide)
-    )
-    (property "Datasheet" "" (at 172.72 124.46 0)
+  (symbol (lib_id "power:GND") (at 121.92 133.35 0) (unit 1)
+    (in_bom yes) (on_board yes) (dnp no) (fields_autoplaced)
+    (property "Reference" "#PWR01" (at 121.92 139.7 0)
+      (effects (font (size 1.27 1.27)) hide)
+    )
+    (property "Value" "GND" (at 121.92 138.43 0)
+      (effects (font (size 1.27 1.27)))
+    )
+    (property "Footprint" "" (at 121.92 133.35 0)
+      (effects (font (size 1.27 1.27)) hide)
+    )
+    (property "Datasheet" "" (at 121.92 133.35 0)
+      (effects (font (size 1.27 1.27)) hide)
+    )
+    (pin "1")
+    (instances
+      (project "EVBuild"
+        (path "/2997cb29-a416-41db-a9e8-1a576f951325"
+          (reference "#PWR01") (unit 1)
+        )
+      )
+    )
+  )
+  (symbol (lib_id "FlyDragon:FlyDragon") (at 214.63 77.47 0) (unit 1)
+    (in_bom yes) (on_board yes) (dnp no) (fields_autoplaced)
+    (property "Reference" "FlyDragon1" (at 212.725 67.31 0)
+      (effects (font (size 1.27 1.27)))
+    )
+    (property "Value" "~" (at 205.74 78.74 0)
+      (effects (font (size 1.27 1.27)))
+    )
+    (property "Footprint" "" (at 205.74 78.74 0)
+      (effects (font (size 1.27 1.27)) hide)
+    )
+    (property "Datasheet" "" (at 205.74 78.74 0)
       (effects (font (size 1.27 1.27)) hide)
     )
@@
         )
       )
+    )
+  )
+  (symbol (lib_id "NCP551:NCP551") (at 36.83 140.97 0) (unit 1)
+    (in_bom yes) (on_board yes) (dnp no) (fields_autoplaced)
+    (property "Reference" "NCP1" (at 38.735 128.27 0)
+      (effects (font (size 1.27 1.27)))
+    )
+    (property "Value" "~" (at 30.48 146.05 0)
+      (effects (font (size 1.27 1.27)))
+    )
+    (property "Footprint" "" (at 30.48 146.05 0)
+      (effects (font (size 1.27 1.27)) hide)
+    )
+    (property "Datasheet" "" (at 30.48 146.05 0)
+      (effects (font (size 1.27 1.27)) hide)
+    )
+    (pin "")
+    (pin "")
+    (pin "")
+    (pin "")
+    (pin "")
+    (instances
+      (project "EVBuild"
+        (path "/2997cb29-a416-41db-a9e8-1a576f951325"
+          (reference "NCP1") (unit 1)
+        )
+      )

Commit message: te other stuff
Parts:
- removed J1: Spark Max PWM, Connector_JST:JST_PH_S4B-PH-K_1x04_P2.00mm_Horizontal, symbol Connector:Conn_01x04_Pin
- removed U2: ~, Package_LGA:Bosch_LGA-14_3x2.5mm_P0.5mm, symbol BMI270:BMI270
- added C1: .1, symbol Device:C
- added C2, C3, C4: 100nF, Capacitor_SMD:C_0201_0603Metric, symbol Device:C
- added J1: Spark Max PWM Pins, Connector_JST:JST_PH_S4B-PH-K_1x04_P2.00mm_Horizontal, symbol Connector:Conn_01x04_Socket
- added R1: 220, symbol Device:R
- added U4: ~, Package_LGA:Bosch_LGA-14_3x2.5mm_P0.5mm, symbol BMI270:BMI270
Connections:
- net GND: now also C1.2, C2.2, C3.2, C4.2, J1.2 (Pin_2), J1.4 (Pin_4), U4.6 (GNDI0), U4.7 (GND)
- net PWM SM2: now reaches U1.12 (IO8)
- net PWM SM2: now also U1.17 (IO9), J1.3 (Pin_3)
- net MOSI: now reaches U1.15 (IO3)
- net MOSI: now also U4.14 (SDx)
- net 3V3: now reaches U1.2 (3V3)
- net 3V3: now also LSF1.3 (A1), LSF1.4 (A2)
- net SCK: now reaches U1.38 (IO2)
- net SCK: now also U4.13 (SCx)
- net CS: now reaches U1.39 (IO1)
- net CS: now also U4.12 (CSB)
- net MISO: now reaches U1.4 (IO4)
- net MISO: now also U4.1 (SDO)
- net INT1: now reaches U1.5 (IO5)
- net INT1: now also U4.4 (INT1)
- net INT2: now reaches U1.6 (IO6)
- net INT2: now also U4.9 (INT2)
- net PWM FlyDragon: now reaches U1.7 (IO7)
- net PWM FlyDragon: now also FlyDragon1. (VCC)
- net +5V: now reaches LSF1.2 (Vref_A)
- net at LSF1.6 (B1): now also FlyDragon1. (VCC)
- net +3.3V: now reaches LSF1.7 (Vref_B)
- net +3.3V: now also R1.1
- net at LSF1.8 (EN): now also C1.1, R1.2
- new net PWM SM1: J1.1 (Pin_1)
- new net VCC: C2.1, C3.1, C4.1, U4.5 (VDDI0), U4.8 (VDD)
- no-connect marks 0 -> 4
Other:
- note added: "ESCs"
- moved on the sheet: FlyDragon1, NCP1
